File: led-strip/hardware/kicad/andon_light_strip.kicad_pcb (KiCad board)
At the start: 2 copper layers, 104 x 21.8 mm, 30 parts

Commit message: chore: update footprint dependencies, added 3d model
Parts:
- D1, D10, D2, D3, D4, D5, D6, D7, D8, D9: footprint Library:worldsemi-WS2812B-2020-V6 -> Sean:worldsemi-WS2812B-2020-V6
- WS-RP2040-Zero1: footprint Library:Waveshare RP2040 Zero -> Sean:Waveshare RP2040 Zero
Changed lines of the file:
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@@
 		(embedded_fonts no)
 	)
-	(footprint "Library:worldsemi-WS2812B-2020-V6"
+	(footprint "Sean:worldsemi-WS2812B-2020-V6"
 		(layer "F.Cu")
 		(at 173.1175 103.035 90)
@@
 		(tags "WS2812B-2020")
 		(property "Reference" "D10"
-			(at 4.285 -0.1175 0)
+			(at 2.07 -3.25 90)
 			(unlocked yes)
 			(layer "F.SilkS")
@@
 				(font
 					(size 1 1)
-					(thickness 0.15)
+					(thickness 0.1)
 				)
 			)
@@
 		)
 		(embedded_fonts no)
+		(model "${MY_3DMODEL_DIR}/LEDs/WS2812-2020.STEP"
+			(offset
+				(xyz 1.7 1.2 0.31)
+			)
+			(scale
+				(xyz 1 1 1)
+			)
+			(rotate
+				(xyz -90 -0 -0)
+			)
+		)
 	)
 	(footprint "Fiducial:Fiducial_1mm_Mask2mm"
@@
 		)
 	)
-	(footprint "Library:Waveshare RP2040 Zero"
+	(footprint "Sean:Waveshare RP2040 Zero"
 		(layer "F.Cu")
 		(at 99.16 110.62 90)
 		(property "Reference" "WS-RP2040-Zero1"
-			(at 10.37 -12.38 0)
+			(at 9 -16 90)
 			(unlocked yes)
 			(layer "F.SilkS")
@@
 		)
 		(property "Value" "Waveshare RP2040 Zero"
-			(at 8.9 -12.15 0)
+			(at 9.5 -14 90)
 			(unlocked yes)
 			(layer "F.Fab")
@@
 		)
 		(fp_text user "${REFERENCE}"
-			(at 5.29 -12 0)
+			(at 9 -12 90)
 			(unlocked yes)
 			(layer "F.Fab")
@@
 			(pinfunction "3V3")
 			(pintype "power_in+no_connect")
-			(zone_connect 0)
 		)
 		(pad "22" thru_hole circle
@@
 			(pinfunction "GND")
 			(pintype "power_in")
-			(zone_connect 2)
 		)
 		(pad "23" thru_hole circle
@@
 		)
 		(embedded_fonts no)
+		(model "${MY_3DMODEL_DIR}/Modules/RP2040-ZERO-WAVESHARE with headers.STEP"
+			(offset
+				(xyz 9 11.75 2.5)
+			)
+			(scale
+				(xyz 1 1 1)
+			)
+			(rotate
+				(xyz 90 -180 -180)
+			)
+		)
 	)
-	(footprint "Library:worldsemi-WS2812B-2020-V6"
+	(footprint "Sean:worldsemi-WS2812B-2020-V6"
 		(layer "F.Cu")
 		(at 143.1175 103.035 90)
@@
 		(tags "WS2812B-2020")
 		(property "Reference" "D5"
-			(at 4.285 -0.6175 0)
+			(at 2.07 -3.25 90)
 			(unlocked yes)
 			(layer "F.SilkS")
@@
 				(font
 					(size 1 1)
-					(thickness 0.15)
+					(thickness 0.1)
 				)
 			)
@@
 		)
 		(fp_text user "${REFERENCE}"
-			(at 1.65 0.6 90)
+			(at 1.4 0.6 90)
 			(layer "F.Fab")
 			(effects
@@
 		)
 		(embedded_fonts no)
+		(model "${MY_3DMODEL_DIR}/LEDs/WS2812-2020.STEP"
+			(offset
+				(xyz 1.7 1.2 0.31)
+			)
+			(scale
+				(xyz 1 1 1)
+			)
+			(rotate
+				(xyz -90 -0 -0)
+			)
+		)
 	)
-	(footprint "Library:worldsemi-WS2812B-2020-V6"
+	(footprint "Sean:worldsemi-WS2812B-2020-V6"
 		(layer "F.Cu")
 		(at 155.1175 103.035 90)
@@
 		(tags "WS2812B-2020")
 		(property "Reference" "D7"
-			(at 4.285 -0.6175 0)
+			(at 2.07 -3.25 90)
 			(unlocked yes)
 			(layer "F.SilkS")
@@
 				(font
 					(size 1 1)
-					(thickness 0.15)
+					(thickness 0.1)
 				)
 			)
@@
 		)
 		(embedded_fonts no)
+		(model "${MY_3DMODEL_DIR}/LEDs/WS2812-2020.STEP"
+			(offset
+				(xyz 1.7 1.2 0.31)
+			)
+			(scale
+				(xyz 1 1 1)
+			)
+			(rotate
+				(xyz -90 -0 -0)
+			)
+		)
 	)
 	(footprint "MountingHole:MountingHole_3.2mm_M3_ISO7380"
@@
 		)
 	)
-	(footprint "Library:worldsemi-WS2812B-2020-V6"
+	(footprint "Sean:worldsemi-WS2812B-2020-V6"
 		(layer "F.Cu")
 		(at 149.1175 103.035 90)
@@
 		(tags "WS2812B-2020")
 		(property "Reference" "D6"
-			(at 4.285 -0.6175 0)
+			(at 2.07 -3.25 90)
 			(unlocked yes)
 			(layer "F.SilkS")
@@
 				(font
 					(size 1 1)
-					(thickness 0.15)
+					(thickness 0.1)
 				)
 			)
@@
 		)
 		(embedded_fonts no)
+		(model "${MY_3DMODEL_DIR}/LEDs/WS2812-2020.STEP"
+			(offset
+				(xyz 1.7 1.2 0.31)
+			)
+			(scale
+				(xyz 1 1 1)
+			)
+			(rotate
+				(xyz -90 -0 -0)
+			)
+		)
 	)
-	(footprint "Library:worldsemi-WS2812B-2020-V6"
+	(footprint "Sean:worldsemi-WS2812B-2020-V6"
 		(layer "F.Cu")
 		(at 167.1175 103.035 90)
@@
 		(tags "WS2812B-2020")
 		(property "Reference" "D9"
-			(at 4.285 -0.6175 0)
+			(at 2.07 -3.25 90)
 			(unlocked yes)
 			(layer "F.SilkS")
@@
 				(font
 					(size 1 1)
-					(thickness 0.15)
+					(thickness 0.1)
 				)
 			)
@@
 		)
 		(embedded_fonts no)
+		(model "${MY_3DMODEL_DIR}/LEDs/WS2812-2020.STEP"
+			(offset
+				(xyz 1.7 1.2 0.31)
+			)
+			(scale
+				(xyz 1 1 1)
+			)
+			(rotate
+				(xyz -90 -0 -0)
+			)
+		)
 	)
 	(footprint "Resistor_SMD:R_0805_2012Metric"
@@
 		)
 	)
-	(footprint "Library:worldsemi-WS2812B-2020-V6"
+	(footprint "Sean:worldsemi-WS2812B-2020-V6"
 		(layer "F.Cu")
 		(at 119.487672 103.035 90)
@@
 		(tags "WS2812B-2020")
 		(property "Reference" "D1"
-			(at 4.285 -0.737672 0)
+			(at 2.07 -3.25 90)
 			(unlocked yes)
 			(layer "F.SilkS")
@@
 				(font
 					(size 1 1)
-					(thickness 0.15)
+					(thickness 0.1)
 				)
 			)
@@
 		)
 		(embedded_fonts no)
+		(model "${MY_3DMODEL_DIR}/LEDs/WS2812-2020.STEP"
+			(offset
+				(xyz 1.7 1.2 0.31)
+			)
+			(scale
+				(xyz 1 1 1)
+			)
+			(rotate
+				(xyz -90 -0 -0)
+			)
+		)
 	)
-	(footprint "Library:worldsemi-WS2812B-2020-V6"
+	(footprint "Sean:worldsemi-WS2812B-2020-V6"
 		(layer "F.Cu")
 		(at 137.1175 103.035 90)
@@
 		(tags "WS2812B-2020")
 		(property "Reference" "D4"
-			(at 4.285 -0.6175 0)
+			(at 2.07 -3.25 90)
 			(unlocked yes)
 			(layer "F.SilkS")
@@
 				(font
 					(size 1 1)
-					(thickness 0.15)
+					(thickness 0.1)
 				)
 			)
@@
 		)
 		(embedded_fonts no)
+		(model "${MY_3DMODEL_DIR}/LEDs/WS2812-2020.STEP"
+			(offset
+				(xyz 1.7 1.2 0.31)
+			)
+			(scale
+				(xyz 1 1 1)
+			)
+			(rotate
+				(xyz -90 -0 -0)
+			)
+		)
 	)
-	(footprint "Library:worldsemi-WS2812B-2020-V6"
+	(footprint "Sean:worldsemi-WS2812B-2020-V6"
 		(layer "F.Cu")
 		(at 125.1175 103.035 90)
@@
 		(tags "WS2812B-2020")
 		(property "Reference" "D2"
-			(at 4.285 -0.6175 0)
+			(at 2.07 -3.25 90)
 			(unlocked yes)
 			(layer "F.SilkS")
@@
 				(font
 					(size 1 1)
-					(thickness 0.15)
+					(thickness 0.1)
 				)
 			)
@@
 		)
 		(embedded_fonts no)
+		(model "${MY_3DMODEL_DIR}/LEDs/WS2812-2020.STEP"
+			(offset
+				(xyz 1.7 1.2 0.31)
+			)
+			(scale
+				(xyz 1 1 1)
+			)
+			(rotate
+				(xyz -90 -0 -0)
+			)
+		)
 	)
 	(footprint "MountingHole:MountingHole_3.2mm_M3_ISO7380"
@@
 		)
 	)
-	(footprint "Library:worldsemi-WS2812B-2020-V6"
+	(footprint "Sean:worldsemi-WS2812B-2020-V6"
 		(layer "F.Cu")
 		(at 131.1175 103.035 90)
@@
 		(tags "WS2812B-2020")
 		(property "Reference" "D3"
-			(at 4.285 -0.6175 0)
+			(at 2.07 -3.25 90)
 			(unlocked yes)
 			(layer "F.SilkS")
@@
 				(font
 					(size 1 1)
-					(thickness 0.15)
+					(thickness 0.1)
 				)
 			)
@@
 		)
 		(embedded_fonts no)
+		(model "${MY_3DMODEL_DIR}/LEDs/WS2812-2020.STEP"
+			(offset
+				(xyz 1.7 1.2 0.31)
+			)
+			(scale
+				(xyz 1 1 1)
+			)
+			(rotate
+				(xyz -90 -0 -0)
+			)
+		)
 	)
 	(footprint "Capacitor_SMD:C_0402_1005Metric"
@@
 		)
 	)
-	(footprint "Library:worldsemi-WS2812B-2020-V6"
+	(footprint "Sean:worldsemi-WS2812B-2020-V6"
 		(layer "F.Cu")
 		(at 161.1175 103.035 90)
@@
 		(tags "WS2812B-2020")
 		(property "Reference" "D8"
-			(at 4.285 -0.6175 0)
+			(at 2.07 -3.25 90)
 			(unlocked yes)
 			(layer "F.SilkS")
@@
 				(font
 					(size 1 1)
-					(thickness 0.15)
+					(thickness 0.1)
 				)
 			)
@@
 		)
 		(embedded_fonts no)
+		(model "${MY_3DMODEL_DIR}/LEDs/WS2812-2020.STEP"
+			(offset
+				(xyz 1.7 1.2 0.31)
+			)
+			(scale
+				(xyz 1 1 1)
+			)
+			(rotate
+				(xyz -90 -0 -0)
+			)
+		)
 	)
 	(gr_arc
